Commit message: Place 6 ZED 2 stereo cameras model (Webots default Camera nodes, without RangeFinder nodes yet) around ego vehicle in simulation world

File: resources/descriptions/EgoVehicle.urdf (robot description, URDF)
Before this commit: robot /home/ayrtom/Computer Vision/dev/FQW_ws/src/surround-view-segbev/resources/descriptions/EgoVehicle.urdf, 13 links, 14 joints
Links:
- added link Eye screw 1; collision cylinder length=0.0009 radius=0.003; collision cylinder length=0.01 radius=0.0018
- added link Eye screw 2; collision cylinder length=0.0009 radius=0.003; collision cylinder length=0.01 radius=0.0018
- added link appearance
- added link appearance_0
- added link appearance_1
- added link appearance_10
- added link appearance_11
- added link appearance_12
- added link appearance_13
- added link appearance_14
- added link appearance_15
- added link appearance_16
- added link appearance_17
- added link appearance_18
- added link appearance_19
- added link appearance_2
- added link appearance_20
- added link appearance_21
- added link appearance_22
- added link appearance_23
- added link appearance_25
- added link appearance_26
- added link appearance_27
- added link appearance_28
- added link appearance_29
- added link appearance_3
- added link appearance_30
- added link appearance_31
- added link appearance_32
- added link appearance_33
- added link appearance_34
- added link appearance_35
- added link appearance_36
- added link appearance_37
- added link appearance_38
- added link appearance_39
- added link appearance_4
- added link appearance_40
- added link appearance_41
- added link appearance_42
- added link appearance_43
- added link appearance_44
- added link appearance_45
- added link appearance_46
- added link appearance_47
- added link appearance_48
- added link appearance_49
- added link appearance_5
- added link appearance_6
- added link appearance_7
- added link appearance_8
- added link appearance_9
- added link camera_front_left
- added link camera_front_right
- added link camera_rear_left
- added link camera_rear_right
- added link torus; collision sphere radius=0.0012; collision sphere radius=0.0012
- added link torus_24; collision sphere radius=0.0012; collision sphere radius=0.0012
Joints:
- removed joint slot_0_rear left wheel_joint
- added joint Eye screw 1_torus_24_joint: type fixed, parent Eye screw 1, child torus_24, origin xyz=-0.0054 0 0 rpy=0 0 0
- added joint Eye screw 2_torus_joint: type fixed, parent Eye screw 2, child torus, origin xyz=-0.0054 0 0 rpy=0 0 0
- added joint base_link_camera_front_left_joint: type fixed, parent base_link, child camera_front_left, origin xyz=3.93794 0.99 0.9125 rpy=-1.570796 0 -0.020796
- added joint base_link_camera_front_right_joint: type fixed, parent base_link, child camera_front_right, origin xyz=3.93773 -0.974 0.9125 rpy=-1.570796 0 -3.120796
- added joint base_link_camera_rear_left_joint: type fixed, parent base_link, child camera_rear_left, origin xyz=4.415817 1.043041 0.77 rpy=-1.570796 0 0.613204
- added joint base_link_camera_rear_right_joint: type fixed, parent base_link, child camera_rear_right, origin xyz=4.427145 -1.02606 0.77 rpy=-1.570796 0 -3.754982
- added joint camera_rear_left_Eye screw 1_joint: type fixed, parent camera_rear_left, child Eye screw 1, origin xyz=-0.122 0 -0.0038 rpy=3.141593 -1.047193 3.141593
- added joint camera_rear_right_Eye screw 2_joint: type fixed, parent camera_rear_right, child Eye screw 2, origin xyz=-0.122 0 -0.0038 rpy=3.141593 -1.047193 3.141593
- added joint slot_50_rear left wheel_joint: type fixed, parent base_link, child rear left wheel, origin xyz=0 0 0 rpy=0 0 0
- added joint torus_24_appearance_25_joint: type fixed, parent torus_24, child appearance_25, origin xyz=0 0 0 rpy=0 0 0
- added joint torus_24_appearance_26_joint: type fixed, parent torus_24, child appearance_26, origin xyz=0 0 0 rpy=0 0 0
- added joint torus_24_appearance_27_joint: type fixed, parent torus_24, child appearance_27, origin xyz=0 0 0 rpy=0 0 0
- added joint torus_24_appearance_28_joint: type fixed, parent torus_24, child appearance_28, origin xyz=0 0 0 rpy=0 0 0
- added joint torus_24_appearance_29_joint: type fixed, parent torus_24, child appearance_29, origin xyz=0 0 0 rpy=0 0 0
- added joint torus_24_appearance_30_joint: type fixed, parent torus_24, child appearance_30, origin xyz=0 0 0 rpy=0 0 0
- added joint torus_24_appearance_31_joint: type fixed, parent torus_24, child appearance_31, origin xyz=0 0 0 rpy=0 0 0
- added joint torus_24_appearance_32_joint: type fixed, parent torus_24, child appearance_32, origin xyz=0 0 0 rpy=0 0 0
- added joint torus_24_appearance_33_joint: type fixed, parent torus_24, child appearance_33, origin xyz=0 0 0 rpy=0 0 0
- added joint torus_24_appearance_34_joint: type fixed, parent torus_24, child appearance_34, origin xyz=0 0 0 rpy=0 0 0
- added joint torus_24_appearance_35_joint: type fixed, parent torus_24, child appearance_35, origin xyz=0 0 0 rpy=0 0 0
- added joint torus_24_appearance_36_joint: type fixed, parent torus_24, child appearance_36, origin xyz=0 0 0 rpy=0 0 0
- added joint torus_24_appearance_37_joint: type fixed, parent torus_24, child appearance_37, origin xyz=0 0 0 rpy=0 0 0
- added joint torus_24_appearance_38_joint: type fixed, parent torus_24, child appearance_38, origin xyz=0 0 0 rpy=0 0 0
- added joint torus_24_appearance_39_joint: type fixed, parent torus_24, child appearance_39, origin xyz=0 0 0 rpy=0 0 0
- added joint torus_24_appearance_40_joint: type fixed, parent torus_24, child appearance_40, origin xyz=0 0 0 rpy=0 0 0
- added joint torus_24_appearance_41_joint: type fixed, parent torus_24, child appearance_41, origin xyz=0 0 0 rpy=0 0 0
- added joint torus_24_appearance_42_joint: type fixed, parent torus_24, child appearance_42, origin xyz=0 0 0 rpy=0 0 0
- added joint torus_24_appearance_43_joint: type fixed, parent torus_24, child appearance_43, origin xyz=0 0 0 rpy=0 0 0
- added joint torus_24_appearance_44_joint: type fixed, parent torus_24, child appearance_44, origin xyz=0 0 0 rpy=0 0 0
- added joint torus_24_appearance_45_joint: type fixed, parent torus_24, child appearance_45, origin xyz=0 0 0 rpy=0 0 0
- added joint torus_24_appearance_46_joint: type fixed, parent torus_24, child appearance_46, origin xyz=0 0 0 rpy=0 0 0
- added joint torus_24_appearance_47_joint: type fixed, parent torus_24, child appearance_47, origin xyz=0 0 0 rpy=0 0 0
- added joint torus_24_appearance_48_joint: type fixed, parent torus_24, child appearance_48, origin xyz=0 0 0 rpy=0 0 0
- added joint torus_24_appearance_49_joint: type fixed, parent torus_24, child appearance_49, origin xyz=0 0 0 rpy=0 0 0
- added joint torus_appearance_0_joint: type fixed, parent torus, child appearance_0, origin xyz=0 0 0 rpy=0 0 0
- added joint torus_appearance_10_joint: type fixed, parent torus, child appearance_10, origin xyz=0 0 0 rpy=0 0 0
- added joint torus_appearance_11_joint: type fixed, parent torus, child appearance_11, origin xyz=0 0 0 rpy=0 0 0
- added joint torus_appearance_12_joint: type fixed, parent torus, child appearance_12, origin xyz=0 0 0 rpy=0 0 0
- added joint torus_appearance_13_joint: type fixed, parent torus, child appearance_13, origin xyz=0 0 0 rpy=0 0 0
- added joint torus_appearance_14_joint: type fixed, parent torus, child appearance_14, origin xyz=0 0 0 rpy=0 0 0
- added joint torus_appearance_15_joint: type fixed, parent torus, child appearance_15, origin xyz=0 0 0 rpy=0 0 0
- added joint torus_appearance_16_joint: type fixed, parent torus, child appearance_16, origin xyz=0 0 0 rpy=0 0 0
- added joint torus_appearance_17_joint: type fixed, parent torus, child appearance_17, origin xyz=0 0 0 rpy=0 0 0
- added joint torus_appearance_18_joint: type fixed, parent torus, child appearance_18, origin xyz=0 0 0 rpy=0 0 0
- added joint torus_appearance_19_joint: type fixed, parent torus, child appearance_19, origin xyz=0 0 0 rpy=0 0 0
- added joint torus_appearance_1_joint: type fixed, parent torus, child appearance_1, origin xyz=0 0 0 rpy=0 0 0
- added joint torus_appearance_20_joint: type fixed, parent torus, child appearance_20, origin xyz=0 0 0 rpy=0 0 0
- added joint torus_appearance_21_joint: type fixed, parent torus, child appearance_21, origin xyz=0 0 0 rpy=0 0 0
- added joint torus_appearance_22_joint: type fixed, parent torus, child appearance_22, origin xyz=0 0 0 rpy=0 0 0
- added joint torus_appearance_23_joint: type fixed, parent torus, child appearance_23, origin xyz=0 0 0 rpy=0 0 0
- added joint torus_appearance_2_joint: type fixed, parent torus, child appearance_2, origin xyz=0 0 0 rpy=0 0 0
- added joint torus_appearance_3_joint: type fixed, parent torus, child appearance_3, origin xyz=0 0 0 rpy=0 0 0
- added joint torus_appearance_4_joint: type fixed, parent torus, child appearance_4, origin xyz=0 0 0 rpy=0 0 0
- added joint torus_appearance_5_joint: type fixed, parent torus, child appearance_5, origin xyz=0 0 0 rpy=0 0 0
- added joint torus_appearance_6_joint: type fixed, parent torus, child appearance_6, origin xyz=0 0 0 rpy=0 0 0
- added joint torus_appearance_7_joint: type fixed, parent torus, child appearance_7, origin xyz=0 0 0 rpy=0 0 0
- added joint torus_appearance_8_joint: type fixed, parent torus, child appearance_8, origin xyz=0 0 0 rpy=0 0 0
- added joint torus_appearance_9_joint: type fixed, parent torus, child appearance_9, origin xyz=0 0 0 rpy=0 0 0
- added joint torus_appearance_joint: type fixed, parent torus, child appearance, origin xyz=0 0 0 rpy=0 0 0
- joint base_link_camera_front_joint: origin xyz=5.26 0.01 0.48 rpy=-1.570796 0 -1.570796 -> xyz=4.12 0.01 1.64 rpy=-1.570796 0 -1.570796
- joint base_link_camera_rear_joint: origin xyz=-1.613499 0.007999 0.555 rpy=-1.570796 0 1.570704 -> xyz=-1.634499 0.008001 0.617 rpy=-1.570796 0 1.570704
- joint left_rear_sensor: origin xyz=0 0.85 0 rpy=0 0.000097 3.14159 -> xyz=0 0.85 0 rpy=0 0 3.14159
- joint right_rear_sensor: origin xyz=0 -0.85 0 rpy=0 -0.000097 0 -> xyz=0 -0.85 0 rpy=0 0 0
