Commit message: Path planning with obstacles avoidance using Nav2 (and probably SLAM Toolbox) frameworks still in progress. Code refactoring (in particular, delete camera_rear_left and camera_rear_right from everywhere for lack of use)

File: resource/descriptions/EgoVehicle.urdf (robot description, URDF)
Before this commit: robot /home/ayrtom/Computer Vision/dev/FQW_ws/src/surround_view_segbev/resource/descriptions/EgoVehicle.urdf, 77 links, 78 joints
Links:
- removed link Eye screw 1
- removed link Eye screw 2
- removed link appearance
- removed link appearance_0
- removed link appearance_1
- removed link appearance_10
- removed link appearance_11
- removed link appearance_12
- removed link appearance_13
- removed link appearance_14
- removed link appearance_15
- removed link appearance_16
- removed link appearance_17
- removed link appearance_18
- removed link appearance_19
- removed link appearance_2
- removed link appearance_20
- removed link appearance_21
- removed link appearance_22
- removed link appearance_23
- removed link appearance_25
- removed link appearance_26
- removed link appearance_27
- removed link appearance_28
- removed link appearance_29
- removed link appearance_3
- removed link appearance_30
- removed link appearance_31
- removed link appearance_32
- removed link appearance_33
- removed link appearance_34
- removed link appearance_35
- removed link appearance_36
- removed link appearance_37
- removed link appearance_38
- removed link appearance_39
- removed link appearance_4
- removed link appearance_40
- removed link appearance_41
- removed link appearance_42
- removed link appearance_43
- removed link appearance_44
- removed link appearance_45
- removed link appearance_46
- removed link appearance_47
- removed link appearance_48
- removed link appearance_49
- removed link appearance_5
- removed link appearance_6
- removed link appearance_7
- removed link appearance_8
- removed link appearance_9
- removed link camera_rear_left
- removed link camera_rear_left_depth
- removed link camera_rear_right
- removed link camera_rear_right_depth
- removed link torus
- removed link torus_24
- added link base_footprint
- added link camera_front_blind
- added link camera_front_blind_depth
- added link compass
- added link gps
- added link imu
Joints:
- removed joint Eye screw 1_torus_24_joint
- removed joint Eye screw 2_torus_joint
- removed joint base_link_camera_rear_left_joint
- removed joint base_link_camera_rear_right_joint
- removed joint camera_rear_left_Eye screw 1_joint
- removed joint camera_rear_left_camera_rear_left_depth_joint
- removed joint camera_rear_right_Eye screw 2_joint
- removed joint camera_rear_right_camera_rear_right_depth_joint
- removed joint slot_50_rear left wheel_joint
- removed joint torus_24_appearance_25_joint
- removed joint torus_24_appearance_26_joint
- removed joint torus_24_appearance_27_joint
- removed joint torus_24_appearance_28_joint
- removed joint torus_24_appearance_29_joint
- removed joint torus_24_appearance_30_joint
- removed joint torus_24_appearance_31_joint
- removed joint torus_24_appearance_32_joint
- removed joint torus_24_appearance_33_joint
- removed joint torus_24_appearance_34_joint
- removed joint torus_24_appearance_35_joint
- removed joint torus_24_appearance_36_joint
- removed joint torus_24_appearance_37_joint
- removed joint torus_24_appearance_38_joint
- removed joint torus_24_appearance_39_joint
- removed joint torus_24_appearance_40_joint
- removed joint torus_24_appearance_41_joint
- removed joint torus_24_appearance_42_joint
- removed joint torus_24_appearance_43_joint
- removed joint torus_24_appearance_44_joint
- removed joint torus_24_appearance_45_joint
- removed joint torus_24_appearance_46_joint
- removed joint torus_24_appearance_47_joint
- removed joint torus_24_appearance_48_joint
- removed joint torus_24_appearance_49_joint
- removed joint torus_appearance_0_joint
- removed joint torus_appearance_10_joint
- removed joint torus_appearance_11_joint
- removed joint torus_appearance_12_joint
- removed joint torus_appearance_13_joint
- removed joint torus_appearance_14_joint
- removed joint torus_appearance_15_joint
- removed joint torus_appearance_16_joint
- removed joint torus_appearance_17_joint
- removed joint torus_appearance_18_joint
- removed joint torus_appearance_19_joint
- removed joint torus_appearance_1_joint
- removed joint torus_appearance_20_joint
- removed joint torus_appearance_21_joint
- removed joint torus_appearance_22_joint
- removed joint torus_appearance_23_joint
- removed joint torus_appearance_2_joint
- removed joint torus_appearance_3_joint
- removed joint torus_appearance_4_joint
- removed joint torus_appearance_5_joint
- removed joint torus_appearance_6_joint
- removed joint torus_appearance_7_joint
- removed joint torus_appearance_8_joint
- removed joint torus_appearance_9_joint
- removed joint torus_appearance_joint
- added joint base_footprint_joint: type fixed, parent base_link, child base_footprint, origin xyz=0 0 0 rpy=0 0 0
- added joint base_link_camera_front_blind_joint: type fixed, parent base_link, child camera_front_blind, origin xyz=5.3622 0.01 0.732 rpy=-1.570796 0.695 -1.570796
- added joint base_link_compass_joint: type fixed, parent base_link, child compass, origin xyz=0 0 0 rpy=0 0 0
- added joint base_link_gps_joint: type fixed, parent base_link, child gps, origin xyz=-0.00613 0 2.3 rpy=0 0 0
- added joint base_link_imu_joint: type fixed, parent base_link, child imu, origin xyz=0 0 0 rpy=0 0 1.5708
- added joint camera_front_blind_camera_front_blind_depth_joint: type fixed, parent camera_front_blind, child camera_front_blind_depth, origin xyz=0 0 0 rpy=0 0 0
- added joint slot_rear left wheel_joint: type fixed, parent base_link, child rear left wheel, origin xyz=0 0 0 rpy=0 0 0
- joint base_link_camera_front_joint: origin xyz=4.12 0.01 1.64 rpy=-1.570796 0 -1.570796 -> xyz=4.12 0.01 1.64 rpy=-1.570796 -0.000005 -1.570796
- joint base_link_camera_front_left_joint: origin xyz=3.93794 0.99 0.9125 rpy=-1.570796 0 -0.020796 -> xyz=1.7379 0.836 2.13828 rpy=-1.570798 0.785396 -0.000802
- joint base_link_camera_front_right_joint: origin xyz=3.93773 -0.974 0.9125 rpy=-1.570796 0 -3.120796 -> xyz=1.7379 -0.817 2.13828 rpy=-1.570795 0.785396 -3.140791
- joint base_link_camera_rear_joint: origin xyz=-1.634499 0.008001 0.617 rpy=-1.570796 0 1.570704 -> xyz=-1.546999 0.007993 2.11955 rpy=-1.570796 0.785398 1.570704

Commit message: Odometry for SLAM Toolbox and Nav2 in progress. Put QoS profiles in separate file

File: resource/descriptions/EgoVehicle.urdf (robot description, URDF)
Before this commit: robot /home/ayrtom/Computer Vision/dev/FQW_ws/src/surround_view_segbev/resource/descriptions/EgoVehicle.urdf, 25 links, 26 joints
Links:
- removed link rear left wheel
- removed link rear right wheel
- added link lidar
- added link rear_left_wheel; collision cylinder length=0.3 radius=0.4; visual cylinder length=0.3 radius=0.4
- added link rear_right_wheel; collision cylinder length=0.3 radius=0.4; visual cylinder length=0.3 radius=0.4
Joints:
- removed joint slot_rear left wheel_joint
- removed joint slot_rear right wheel_joint
- added joint base_link_lidar_joint: type fixed, parent base_link, child lidar, origin xyz=4.6 0 1.14 rpy=0 0 0
- added joint rear_left_wheel_joint: type fixed, parent base_link, child rear_left_wheel, origin xyz=0 0 0 rpy=0 0 0
- added joint rear_right_wheel_joint: type fixed, parent base_link, child rear_right_wheel, origin xyz=0 0 0 rpy=0 0 0
- joint base_link_imu_joint: origin xyz=0 0 0 rpy=0 0 1.5708 -> xyz=0 0 0 rpy=0 0 0
- joint left_rear_sensor: child rear left wheel -> rear_left_wheel
- joint right_rear_sensor: child rear right wheel -> rear_right_wheel

Commit message: Develop tool called BEVFormer for more visual surround view image formation. Major code refactoring

File: resource/descriptions/EgoVehicle.urdf (robot description, URDF)
Before this commit: robot /home/ayrtom/Computer Vision/dev/FQW_ws/src/surround_view_segbev/resource/descriptions/EgoVehicle.urdf, 26 links, 27 joints
Links:
- added link accelerometer
- added link gyroscope
Joints:
- added joint base_link_accelerometer_joint: type fixed, parent base_link, child accelerometer, origin xyz=0 0 0 rpy=0 0 0
- added joint base_link_gyroscope_joint: type fixed, parent base_link, child gyroscope, origin xyz=0 0 0 rpy=0 0 0
- joint base_link_camera_front_blind_joint: origin xyz=5.3622 0.01 0.732 rpy=-1.570796 0.695 -1.570796 -> xyz=5.3622 0.01 0.732 rpy=0 0 0

Commit message: Add support for rear lidar and it's point cloud merge with front lidar data. Minor folders restructure and code refactoring

File: resource/descriptions/EgoVehicle.urdf (robot description, URDF)
Before this commit: robot /home/ayrtom/ROS2/dev/FQW_ws/src/surround_view_segbev/resource/descriptions/EgoVehicle.urdf, 28 links, 29 joints
Links:
- removed link lidar
- added link lidar_front
- added link lidar_rear
Joints:
- removed joint base_link_lidar_joint
- added joint base_link_lidar_front_joint: type fixed, parent base_link, child lidar_front, origin xyz=4.6 0 1.14 rpy=0 0 0
- added joint base_link_lidar_rear_joint: type fixed, parent base_link, child lidar_rear, origin xyz=-1.67 0.000005 0.14 rpy=0 0 3.1415
